File: Pro/PCB/Lily58_Pro.kicad_pcb (KiCad board)
At the start: 2 copper layers, 142.5 x 112.3 mm, 63 parts, among them J1 OLED, J2 TRRS, SW1 SW_PUSH, SW10 SW_PUSH, SW11 SW_PUSH, SW12 SW_PUSH, SW13 SW_PUSH, SW14 SW_PUSH, SW15 SW_PUSH, SW16 SW_PUSH, SW17 SW_PUSH, SW18 SW_PUSH, SW19 SW_PUSH, SW2 SW_PUSH, SW20 SW_PUSH, SW21 SW_PUSH, SW22 SW_PUSH, SW23 SW_PUSH, SW24 SW_PUSH, SW25 SW_PUSH, SW26 SW_PUSH, SW27 SW_PUSH, SW28 SW_PUSH, SW29 SW_PUSH, SW3 SW_PUSH, SW4 SW_PUSH, SW5 SW_PUSH, SW6 SW_PUSH, SW7 SW_PUSH, SW8 SW_PUSH, SW9 SW_PUSH

Commit message: Remove old files
Routing:
- net row4: track 125.1 -> 123.0 mm
Changed lines of the file:
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@@
       (sketchpadsonfab false)
       (subtractmaskfromsilk false)
-      (outputformat 1)
+      (outputformat 3)
       (mirror false)
       (drillshape 0)
@@
     (stroke (width 0.2) (type solid)) (layer "Edge.Cuts"))
   (dimension (type aligned) (layer "Eco1.User")
-    (pts (xy 83.010647 143.990685) (xy 83.010647 36.990685))
-    (height -3)
-    (gr_text "107.0000 mm" (at 78.210647 90.490685 90) (layer "Eco1.User")
-      (effects (font (size 1.5 1.5) (thickness 0.3)))
+    (pts (xy 83 37) (xy 83 150))
+    (height 3)
+    (gr_text "113.0000 mm" (at 78.2 93.5 90) (layer "Eco1.User")
+      (effects (font (size 1.5 1.5) (thickness 0.3) bold))
     )
-    (format (prefix "") (suffix "") (units 2) (units_format 1) (precision 4))
+    (format (prefix "") (suffix "") (units 3) (units_format 1) (precision 4))
     (style (thickness 0.3) (arrow_length 1.27) (text_position_mode 0) (extension_height 0.58642) (extension_offset 0) keep_text_aligned)
   )
@@
   (segment (start 116.340979 125.391489) (end 116.340979 125.340021) (width 0.25) (layer "F.Cu") (net 1))
   (segment (start 110.998 69.215) (end 110.617 68.834) (width 0.25) (layer "F.Cu") (net 1))
+  (segment (start 116.340979 118.364) (end 116.340979 117.570982) (width 0.25) (layer "F.Cu") (net 1))
   (segment (start 106.840979 103.344021) (end 107.95 102.235) (width 0.25) (layer "F.Cu") (net 1))
   (segment (start 110.998 90.302) (end 110.998 69.215) (width 0.25) (layer "F.Cu") (net 1))
@@
   (segment (start 128.35 118) (end 130.6 115.75) (width 0.25) (layer "F.Cu") (net 1))
   (segment (start 105.887295 67.57973) (end 105.496295 67.57973) (width 0.25) (layer "F.Cu") (net 1))
-  (segment (start 123.317 118.364) (end 127.986 118.364) (width 0.25) (layer "F.Cu") (net 1))
   (segment (start 105.887295 67.97073) (end 105.887295 67.57973) (width 0.25) (layer "F.Cu") (net 1))
+  (segment (start 127.986 118.364) (end 116.340979 118.364) (width 0.25) (layer "F.Cu") (net 1))
   (segment (start 147.35 115.75) (end 148.6 114.5) (width 0.25) (layer "F.Cu") (net 1))
   (segment (start 106.553 94.771) (end 106.553 94.747) (width 0.25) (layer "F.Cu") (net 1))
   (segment (start 110.617 68.834) (end 106.750565 68.834) (width 0.25) (layer "F.Cu") (net 1))
-  (segment (start 116.340979 125.340021) (end 123.317 118.364) (width 0.25) (layer "F.Cu") (net 1))
   (segment (start 148.6 114.5) (end 165.2 114.5) (width 0.25) (layer "F.Cu") (net 1))
   (segment (start 165.2 114.5) (end 166.45 115.75) (width 0.25) (layer "F.Cu") (net 1))
@@
   (segment (start 106.840979 108.937007) (end 106.840979 103.344021) (width 0.25) (layer "F.Cu") (net 1))
   (segment (start 107.95 96.168) (end 106.553 94.771) (width 0.25) (layer "F.Cu") (net 1))
-  (segment (start 127.986 118.364) (end 128.35 118) (width 0.25) (layer "F.Cu") (net 1))
+  (segment (start 128.35 118) (end 127.986 118.364) (width 0.25) (layer "F.Cu") (net 1))
   (segment (start 121.158 57.785) (end 119.693 59.25) (width 0.25) (layer "F.Cu") (net 2))
   (segment (start 178.436 59.436) (end 187.198 59.436) (width 0.25) (layer "F.Cu") (net 2))
