File: Pro/PCB/Lily58_Pro.kicad_pcb (KiCad board)
At the start: 2 copper layers, 142.5 x 112.3 mm, 63 parts, among them J1 OLED, J2 TRRS, SW1 SW_PUSH, SW10 SW_PUSH, SW11 SW_PUSH, SW12 SW_PUSH, SW13 SW_PUSH, SW14 SW_PUSH, SW15 SW_PUSH, SW16 SW_PUSH, SW17 SW_PUSH, SW18 SW_PUSH, SW19 SW_PUSH, SW2 SW_PUSH, SW20 SW_PUSH, SW21 SW_PUSH, SW22 SW_PUSH, SW23 SW_PUSH, SW24 SW_PUSH, SW25 SW_PUSH, SW26 SW_PUSH, SW27 SW_PUSH, SW28 SW_PUSH, SW29 SW_PUSH, SW3 SW_PUSH, SW4 SW_PUSH, SW5 SW_PUSH, SW6 SW_PUSH, SW7 SW_PUSH, SW8 SW_PUSH, SW9 SW_PUSH

Commit message: Production run
Parts:
- removed JP13, JP14, JP15, JP16: ~, Lily58-footprint:Jumper_arrow
- removed Pw2: SW_SPDT, open-project:SWITCH_ALPS_SSSS8
- BT1: footprint Connector_JST:JST_PH_S2B-PH-K_1x02_P2.00mm_Horizontal -> Lily58_Pro-footprint:Battery
- Pw1: footprint open-project:SWITCH_ALPS_SSSS8 -> Lily58-footprint:Power_Switch
- RSW1: footprint Lily58-footprint:TACT_SWITCH_TVBP06 -> Lily58-footprint:Reset_Button
- moved J1 5.24 mm to (100.7, 74.6)
- moved JP10 3.24 mm to (86.2, 74.7)
- moved JP12 3.24 mm to (86.2, 74.7)
- moved JP11 3.23 mm to (88.7, 74.7)
- moved JP9 3.23 mm to (88.7, 74.7)
- moved BT1 1.81 mm to (87.1, 79.1)
- moved JP3 0.21 mm to (98.1, 72.0)
- moved JP7 0.21 mm to (98.1, 72.0)
- moved JP2 0.18 mm to (103.2, 72.0)
- moved JP6 0.18 mm to (103.2, 72.0)
- moved JP4 0.16 mm to (95.6, 72.0)
- moved JP8 0.16 mm to (95.6, 72.0)
- moved JP1 0.12 mm to (105.8, 72.0)
- moved JP5 0.12 mm to (105.8, 72.0)
- moved Pw1 0.09 mm to (84.7, 57.8)
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Connections:
- BT1 pad 1: Net-(BT1--) -> Net-(BT1-+)
- BT1 pad 2: Net-(BT1-+) -> Net-(BT1--)
- ENC1 pad A: Net-(ENC1-PadA) -> encA
- ENC1 pad B: Net-(ENC1-PadB) -> encB
Routing:
- net col3: track 82.1 -> 148.4 mm
- net GND: track 89.8 -> 104.1 mm, vias 2 -> 3
- net Net-(ENC1-PadB): track 12.7 -> 0.00 mm, vias 1 -> 0
- net RESET: track 27.9 -> 39.5 mm
- net encB: track 40.3 -> 50.7 mm, vias 1 -> 0
- net Net-(ENC1-PadA): track 8.70 -> 0.00 mm, vias 1 -> 0
- net BAT_POS: track 19.8 -> 25.5 mm
- net Net-(BT1--): track 10.7 -> 6.82 mm
- net encA: track 44.8 -> 48.3 mm, vias 2 -> 0
- net Net-(BT1-+): track 9.79 -> 6.92 mm
- net SCL: track 37.1 -> 35.0 mm
- net RAW: track 27.3 -> 28.8 mm
- net row4: track 123.0 -> 121.9 mm
- net SDA: track 52.4 -> 51.7 mm
- net CS: track 65.0 -> 64.3 mm
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Other:
- board size 142.5 x 112.3 mm -> 142.5 x 111.4 mm

Commit message: Cleanup
Parts:
- BT1: footprint Lily58_Pro-footprint:Battery -> Lily58-footprint:Battery
- D1: value Lily58-cache:D -> Lily58:D
- ENC1: footprint Rotary_Encoder:RotaryEncoder_Alps_EC11E-Switch_Vertical_H20mm -> Lily58-footprint:RotaryEncoder_EC11
- SW19, SW20, SW21, SW22, SW23, SW24: footprint Lily58-footprint:MX_Choc_Hotswap_bottom_diode -> Lily58-footprint:MX_Choc_Hotswap_left_diode
- moved ENC1 7.90 mm to (96.3, 95.8)
- moved J1 5.08 mm to (95.6, 74.6)
Routing:
- net Net-(SW24-A): track 4.00 -> 0.00 mm
- net row3: track 154.0 -> 156.5 mm
- net row4: track 121.9 -> 124.4 mm
- net col0: track 192.9 -> 191.8 mm

Commit message: Small fixes
Connections:
- J2 pad 1: RAW -> unconnected-(J2-Pad1)
- J2 pad 2: unconnected-(J2-Pad2) -> RAW
- J2 pad 3: GND -> unconnected-(J2-Pad3)
- J2 pad 4: unconnected-(J2-Pad4) -> GND
Routing:
- net GND: track 104.1 -> 90.6 mm, vias 3 -> 2
- net unconnected-(J2-Pad3): track 0.00 -> 5.95 mm
- net unconnected-(J2-Pad2): track 5.95 -> 0.00 mm
- net unconnected-(J2-Pad1): track 0.00 -> 5.30 mm
- net unconnected-(J2-Pad4): track 2.45 -> 0.00 mm
- net RESET: track 39.5 -> 38.6 mm, vias 2 -> 0
- net BAT_POS: track 25.5 -> 26.3 mm
- net RAW: track 28.8 -> 29.5 mm
