File: Pro/PCB/Lily58_Pro.kicad_sch (KiCad schematic)
At the start: 86 parts, among them J1 OLED, J2 4PIN, SW1 SW_PUSH, SW10 SW_PUSH, SW11 SW_PUSH, SW12 SW_PUSH, SW13 SW_PUSH, SW14 SW_PUSH, SW15 SW_PUSH, SW16 SW_PUSH, SW17 SW_PUSH, SW18 SW_PUSH, SW19 SW_PUSH, SW2 SW_PUSH, SW20 SW_PUSH, SW21 SW_PUSH, SW22 SW_PUSH, SW23 SW_PUSH, SW24 SW_PUSH, SW25 SW_PUSH, SW26 SW_PUSH, SW27 SW_PUSH, SW28 SW_PUSH, SW29 SW_PUSH, SW3 SW_PUSH, SW4 SW_PUSH, SW5 SW_PUSH, SW6 SW_PUSH, SW7 SW_PUSH, SW8 SW_PUSH, SW9 SW_PUSH, U1 NiceNano

Commit message: v2
Parts:
- removed D1, D10, D11, D12, D13, D14, D15, D16, D17, D18, D19, D2, D20, D21, D22, D23, D24, D25, D26, D27, D28, D29, D3, D4, D5, D6, D7, D8, D9: D, Lily58-footprint:Diode_SOD123, symbol Lily58_Pro-rescue:D-Lily58-cache
- removed JP3, JP8: Jumper_NO_Small, Lily58-footprint:Jumper, symbol Lily58_Pro-rescue:Jumper_NO_Small-Device
- removed TH1, TH2: HOLE, Lily58-footprint:M2_HOLE_PCB, symbol Lily58_Pro-rescue:HOLE-Lily58-cache
- removed TH3, TH4, TH5, TH6, TH7: HOLE, Lily58-footprint:HOLE_M2_TH, symbol Lily58_Pro-rescue:HOLE-Lily58-cache
- added D1: Lily58-cache:D, Lily58-footprint:Diode_SOD123, symbol Lily58-cache:Lily58-cache{colon}D
- added ENC1: RotaryEncoder_Switch, Rotary_Encoder:RotaryEncoder_Alps_EC11E-Switch_Vertical_H20mm, symbol Device:RotaryEncoder_Switch
- added JP13, JP14, JP15, JP16: ~, Lily58-footprint:Jumper_arrow, symbol Lily58-cache:Device{colon}Jumper_NO_Small
- J1: footprint Lily58-footprint:OLED_4Pin -> Lily58-footprint:NiceView_5Pin; symbol Lily58_Pro-rescue:OLED-Lily58-cache -> Lily58_Pro-rescue:NiceView
- J2: value 4PIN -> TRRS
- JP1, JP2: value Jumper_NO_Small -> ~; footprint Lily58-footprint:Jumper -> Lily58-footprint:Jumper_arrow
- JP10: renamed from JP12; value Device:Jumper_NO_Small -> ~; footprint Lily58-footprint:Jumper -> Lily58-footprint:Jumper_arrow
- JP11: renamed from JP13; value Device:Jumper_NO_Small -> ~; footprint Lily58-footprint:Jumper -> Lily58-footprint:Jumper_arrow
- JP12: renamed from JP14; value Device:Jumper_NO_Small -> ~; footprint Lily58-footprint:Jumper -> Lily58-footprint:Jumper_arrow
- JP3: renamed from JP4; value Jumper_NO_Small -> ~; footprint Lily58-footprint:Jumper -> Lily58-footprint:Jumper_arrow
- JP4: renamed from JP5; value Jumper_NO_Small -> ~; footprint Lily58-footprint:Jumper -> Lily58-footprint:Jumper_arrow
- JP5: renamed from JP6; value JP6 -> ~; footprint Lily58-footprint:Jumper -> Lily58-footprint:Jumper_arrow
- JP6: renamed from JP7; value Jumper_NO_Small -> ~; footprint Lily58-footprint:Jumper -> Lily58-footprint:Jumper_arrow
- JP7: renamed from JP9; value Jumper_NO_Small -> ~; footprint Lily58-footprint:Jumper -> Lily58-footprint:Jumper_arrow
- JP8: renamed from JP10; value Jumper_NO_Small -> ~; footprint Lily58-footprint:Jumper -> Lily58-footprint:Jumper_arrow
- JP9: renamed from JP11; value Device:Jumper_NO_Small -> ~; footprint Lily58-footprint:Jumper -> Lily58-footprint:Jumper_arrow
- MCU1: renamed from U1; footprint Lily58-footprint:ProMicro_rev2 -> Lily58-footprint:ProMicro_rev3; symbol Lily58-cache:Lily58-cache{colon}ProMicro_2 -> ScottoKeebs:MCU_Nice_Nano_V2
- SW1: footprint Lily58-footprint:MX_Choc_Hotswap -> Lily58-footprint:MX_Choc_Hotswap_bottom_diode; symbol Lily58_Pro-rescue:SW_PUSH-Lily58-cache -> Lily58_Pro-rescue:SW_PUSH-Diode-Lily58
- SW10: renamed from SW17; footprint Lily58-footprint:MX_Choc_Hotswap -> Lily58-footprint:MX_Choc_Hotswap_bottom_diode; symbol Lily58_Pro-rescue:SW_PUSH-Lily58-cache -> Lily58_Pro-rescue:SW_PUSH-Diode-Lily58
- SW11: renamed from SW22; footprint Lily58-footprint:MX_Choc_Hotswap -> Lily58-footprint:MX_Choc_Hotswap_bottom_diode; symbol Lily58_Pro-rescue:SW_PUSH-Lily58-cache -> Lily58_Pro-rescue:SW_PUSH-Diode-Lily58
- SW12: renamed from SW27; footprint Lily58-footprint:MX_Choc_Hotswap -> Lily58-footprint:MX_Choc_Hotswap_bottom_diode; symbol Lily58_Pro-rescue:SW_PUSH-Lily58-cache -> Lily58_Pro-rescue:SW_PUSH-Diode-Lily58
- SW13: renamed from SW3; footprint Lily58-footprint:MX_Choc_Hotswap -> Lily58-footprint:MX_Choc_Hotswap_bottom_diode; symbol Lily58_Pro-rescue:SW_PUSH-Lily58-cache -> Lily58_Pro-rescue:SW_PUSH-Diode-Lily58
- SW14: renamed from SW8; footprint Lily58-footprint:MX_Choc_Hotswap -> Lily58-footprint:MX_Choc_Hotswap_bottom_diode; symbol Lily58_Pro-rescue:SW_PUSH-Lily58-cache -> Lily58_Pro-rescue:SW_PUSH-Diode-Lily58
- SW15: renamed from SW13; footprint Lily58-footprint:MX_Choc_Hotswap -> Lily58-footprint:MX_Choc_Hotswap_bottom_diode; symbol Lily58_Pro-rescue:SW_PUSH-Lily58-cache -> Lily58_Pro-rescue:SW_PUSH-Diode-Lily58
- SW16: renamed from SW18; footprint Lily58-footprint:MX_Choc_Hotswap -> Lily58-footprint:MX_Choc_Hotswap_bottom_diode; symbol Lily58_Pro-rescue:SW_PUSH-Lily58-cache -> Lily58_Pro-rescue:SW_PUSH-Diode-Lily58
- SW17: renamed from SW23; footprint Lily58-footprint:MX_Choc_Hotswap -> Lily58-footprint:MX_Choc_Hotswap_bottom_diode; symbol Lily58_Pro-rescue:SW_PUSH-Lily58-cache -> Lily58_Pro-rescue:SW_PUSH-Diode-Lily58
- SW18: renamed from SW28; footprint Lily58-footprint:MX_Choc_Hotswap -> Lily58-footprint:MX_Choc_Hotswap_bottom_diode; symbol Lily58_Pro-rescue:SW_PUSH-Lily58-cache -> Lily58_Pro-rescue:SW_PUSH-Diode-Lily58
- SW19: renamed from SW4; footprint Lily58-footprint:MX_Choc_Hotswap -> Lily58-footprint:MX_Choc_Hotswap_bottom_diode; symbol Lily58_Pro-rescue:SW_PUSH-Lily58-cache -> Lily58_Pro-rescue:SW_PUSH-Diode-Lily58
- SW2: renamed from SW6; footprint Lily58-footprint:MX_Choc_Hotswap -> Lily58-footprint:MX_Choc_Hotswap_bottom_diode; symbol Lily58_Pro-rescue:SW_PUSH-Lily58-cache -> Lily58_Pro-rescue:SW_PUSH-Diode-Lily58
- SW20: renamed from SW9; footprint Lily58-footprint:MX_Choc_Hotswap -> Lily58-footprint:MX_Choc_Hotswap_bottom_diode; symbol Lily58_Pro-rescue:SW_PUSH-Lily58-cache -> Lily58_Pro-rescue:SW_PUSH-Diode-Lily58
- SW21: renamed from SW14; footprint Lily58-footprint:MX_Choc_Hotswap -> Lily58-footprint:MX_Choc_Hotswap_bottom_diode; symbol Lily58_Pro-rescue:SW_PUSH-Lily58-cache -> Lily58_Pro-rescue:SW_PUSH-Diode-Lily58
- SW22: renamed from SW19; footprint Lily58-footprint:MX_Choc_Hotswap -> Lily58-footprint:MX_Choc_Hotswap_bottom_diode; symbol Lily58_Pro-rescue:SW_PUSH-Lily58-cache -> Lily58_Pro-rescue:SW_PUSH-Diode-Lily58
- SW23: renamed from SW24; footprint Lily58-footprint:MX_Choc_Hotswap -> Lily58-footprint:MX_Choc_Hotswap_bottom_diode; symbol Lily58_Pro-rescue:SW_PUSH-Lily58-cache -> Lily58_Pro-rescue:SW_PUSH-Diode-Lily58
- SW24: renamed from SW29; footprint Lily58-footprint:MX_Choc_Hotswap -> Lily58-footprint:MX_Choc_Hotswap_bottom_diode; symbol Lily58_Pro-rescue:SW_PUSH-Lily58-cache -> Lily58_Pro-rescue:SW_PUSH-Diode-Lily58
- SW25: renamed from SW5; footprint Lily58-footprint:MX_Choc_Hotswap -> Lily58-footprint:MX_Choc_Hotswap_right_diode; symbol Lily58_Pro-rescue:SW_PUSH-Lily58-cache -> Lily58_Pro-rescue:SW_PUSH-Diode-Lily58
- SW26: renamed from SW10; footprint Lily58-footprint:MX_Choc_Hotswap -> Lily58-footprint:MX_Choc_Hotswap_right_diode; symbol Lily58_Pro-rescue:SW_PUSH-Lily58-cache -> Lily58_Pro-rescue:SW_PUSH-Diode-Lily58
- SW27: renamed from SW15; footprint Lily58-footprint:MX_Choc_Hotswap -> Lily58-footprint:MX_Choc_Hotswap_top_diode; symbol Lily58_Pro-rescue:SW_PUSH-Lily58-cache -> Lily58_Pro-rescue:SW_PUSH-Diode-Lily58
- SW28: renamed from SW20; footprint Lily58-footprint:MX_Choc_Hotswap -> Lily58-footprint:MX_Choc_Hotswap_top_diode; symbol Lily58_Pro-rescue:SW_PUSH-Lily58-cache -> Lily58_Pro-rescue:SW_PUSH-Diode-Lily58
- SW29: renamed from SW25; footprint Lily58-footprint:MX_Choc_Hotswap -> Lily58-footprint:MX_Choc_Hotswap_top_diode; symbol Lily58_Pro-rescue:SW_PUSH-Lily58-cache -> Lily58_Pro-rescue:SW_PUSH-Diode-Lily58
- SW3: renamed from SW11; footprint Lily58-footprint:MX_Choc_Hotswap -> Lily58-footprint:MX_Choc_Hotswap_bottom_diode; symbol Lily58_Pro-rescue:SW_PUSH-Lily58-cache -> Lily58_Pro-rescue:SW_PUSH-Diode-Lily58
- SW4: renamed from SW16; footprint Lily58-footprint:MX_Choc_Hotswap -> Lily58-footprint:MX_Choc_Hotswap_bottom_diode; symbol Lily58_Pro-rescue:SW_PUSH-Lily58-cache -> Lily58_Pro-rescue:SW_PUSH-Diode-Lily58
- SW5: renamed from SW21; footprint Lily58-footprint:MX_Choc_Hotswap -> Lily58-footprint:MX_Choc_Hotswap_bottom_diode; symbol Lily58_Pro-rescue:SW_PUSH-Lily58-cache -> Lily58_Pro-rescue:SW_PUSH-Diode-Lily58
- SW6: renamed from SW26; footprint Lily58-footprint:MX_Choc_Hotswap -> Lily58-footprint:MX_Choc_Hotswap_bottom_diode; symbol Lily58_Pro-rescue:SW_PUSH-Lily58-cache -> Lily58_Pro-rescue:SW_PUSH-Diode-Lily58
- SW7: renamed from SW2; footprint Lily58-footprint:MX_Choc_Hotswap -> Lily58-footprint:MX_Choc_Hotswap_bottom_diode; symbol Lily58_Pro-rescue:SW_PUSH-Lily58-cache -> Lily58_Pro-rescue:SW_PUSH-Diode-Lily58
- SW8: renamed from SW7; footprint Lily58-footprint:MX_Choc_Hotswap -> Lily58-footprint:MX_Choc_Hotswap_bottom_diode; symbol Lily58_Pro-rescue:SW_PUSH-Lily58-cache -> Lily58_Pro-rescue:SW_PUSH-Diode-Lily58
- SW9: renamed from SW12; footprint Lily58-footprint:MX_Choc_Hotswap -> Lily58-footprint:MX_Choc_Hotswap_bottom_diode; symbol Lily58_Pro-rescue:SW_PUSH-Lily58-cache -> Lily58_Pro-rescue:SW_PUSH-Diode-Lily58
Connections:
- net GND: now also ENC1.C
- net VCC: now also J1.3 (P3)
- net col0: now also SW29.1
- net col1: now also SW28.1; no longer SW29.1
- net col2: now also SW27.1; no longer SW28.1
- net col3: now also SW26.1; no longer SW27.1
- net col4: now also SW25.1; no longer SW26.1
- net col5: now also ENC1.S2; no longer SW25.1
- net row0: now also SW1.3, SW2.3, SW3.3, SW4.3, SW5.3, SW6.3
- net row1: now also SW10.3, SW11.3, SW12.3, SW7.3, SW8.3, SW9.3
- net row2: now also SW13.3, SW14.3, SW15.3, SW16.3, SW17.3, SW18.3
- net row3: now also SW19.3, SW20.3, SW21.3, SW22.3, SW23.3, SW24.3
- net row4: now also SW25.3, SW26.3, SW27.3, SW28.3, SW29.3, D1.1 (K)
- net encB: now reaches MCU1.19 (D20)
- net encB: now also JP13.2, JP16.2
- net encA: now reaches MCU1.20 (D21)
- net encA: now also JP14.2, JP15.2
- net POWER renamed RAW
- new net: ENC1.B, JP13.1, JP15.1
- new net: ENC1.A, JP14.1, JP16.1
- new net: D1.2 (A), ENC1.S1
Other:
- moved on the sheet: JP7, JP8

Commit message: Production run
Parts:
- removed JP13, JP14, JP15, JP16: ~, Lily58-footprint:Jumper_arrow, symbol Lily58-cache:Device{colon}Jumper_NO_Small
- removed Pw2: SW_SPDT, open-project:SWITCH_ALPS_SSSS8, symbol Switch:SW_SPDT
- BT1: footprint Connector_JST:JST_PH_S2B-PH-K_1x02_P2.00mm_Horizontal -> Lily58_Pro-footprint:Battery
- Pw1: footprint open-project:SWITCH_ALPS_SSSS8 -> Lily58-footprint:Power_Switch
- RSW1: footprint Lily58-footprint:TACT_SWITCH_TVBP06 -> Lily58-footprint:Reset_Button
Connections:
- net encA: now also ENC1.A
- net encB: now also ENC1.B
- net at JP10.1, JP12.1: now also BT1.2 (-); no longer BT1.1 (-)
- net at JP11.1, JP9.1: now also BT1.1 (+); no longer BT1.2 (+)
Other:
- moved on the sheet: D1, ENC1, Pw1, RSW1

Commit message: Cleanup
Parts:
- BT1: footprint Lily58_Pro-footprint:Battery -> Lily58-footprint:Battery
- D1: value Lily58-cache:D -> Lily58:D; symbol Lily58-cache:Lily58-cache{colon}D -> Lily58:D
- ENC1: footprint Rotary_Encoder:RotaryEncoder_Alps_EC11E-Switch_Vertical_H20mm -> Lily58-footprint:RotaryEncoder_EC11
- J1: symbol Lily58_Pro-rescue:NiceView -> Lily58:NiceView
- J2: symbol Lily58_Pro-rescue:MJ-4PP-9-Lily58-cache -> Lily58:MJ-4PP-9
- JP1, JP5, JP9: symbol Lily58-cache:Device{colon}Jumper_NO_Small -> Lily58:Jumper_NO_Small
- JP10, JP11, JP12, JP2, JP3, JP4, JP6, JP7, JP8: symbol Lily58_Pro-rescue:Jumper_NO_Small-Device -> Lily58:Jumper_NO_Small
- MCU1: symbol ScottoKeebs:MCU_Nice_Nano_V2 -> Lily58:ProMicro_2
- RSW1: symbol Lily58_Pro-rescue:SW_RST-Lily58-cache -> Lily58:SW_RST
- SW1, SW10, SW11, SW12, SW13, SW14, SW15, SW16, SW17, SW18, SW2, SW25, SW26, SW27, SW28, SW29, SW3, SW4, SW5, SW6, SW7, SW8, SW9: symbol Lily58_Pro-rescue:SW_PUSH-Diode-Lily58 -> Lily58:SW_PUSH-Diode
- SW19, SW20, SW21, SW22, SW23, SW24: footprint Lily58-footprint:MX_Choc_Hotswap_bottom_diode -> Lily58-footprint:MX_Choc_Hotswap_left_diode; symbol Lily58_Pro-rescue:SW_PUSH-Diode-Lily58 -> Lily58:SW_PUSH-Diode

Commit message: Small fixes
Connections:
- net GND: now also J2.4; no longer J2.3
- net RAW: now also J2.2; no longer J2.1
Changed lines of the file:
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@@
-    )
-  )
-  (global_label "RESET" (shape input) (at 69.85 93.98 0)
-    (effects (font (size 1.27 1.27)) (justify left))
-    (property "Intersheetrefs" "${INTERSHEET_REFS}" (at 69.85 93.98 0)
-      (effects (font (size 1.27 1.27)) hide)
     )
   )
@@
     (effects (font (size 1.27 1.27)) (justify right))
     (property "Intersheetrefs" "${INTERSHEET_REFS}" (at 64.77 53.34 0)
+      (effects (font (size 1.27 1.27)) hide)
+    )
+  )
+  (global_label "RESET" (shape input) (at 69.85 93.98 0)
+    (effects (font (size 1.27 1.27)) (justify left))
+    (property "Intersheetrefs" "${INTERSHEET_REFS}" (at 69.85 93.98 0)
       (effects (font (size 1.27 1.27)) hide)
     )
@@
     )
   )
+  (global_label "RAW" (shape input) (at 80.01 113.03 0) (fields_autoplaced)
+    (effects (font (size 1.27 1.27)) (justify left))
+    (property "Intersheetrefs" "${INTERSHEET_REFS}" (at 86.151 113.03 0)
+      (effects (font (size 1.27 1.27)) (justify left) hide)
+    )
+  )
   (global_label "row4" (shape input) (at 133.35 130.81 180)
     (effects (font (size 1.27 1.27)) (justify right))
@@
     (property "Intersheetrefs" "${INTERSHEET_REFS}" (at 220.98 57.15 0)
       (effects (font (size 1.27 1.27)) hide)
-    )
-  )
-  (global_label "RAW" (shape input) (at 80.01 110.49 0) (fields_autoplaced)
-    (effects (font (size 1.27 1.27)) (justify left))
-    (property "Intersheetrefs" "${INTERSHEET_REFS}" (at 86.151 110.49 0)
-      (effects (font (size 1.27 1.27)) (justify left) hide)
     )
   )
@@
     )
   )
-  (symbol (lib_id "power:GND") (at 80.01 115.57 0) (unit 1)
-    (in_bom yes) (on_board yes) (dnp no)
-    (property "Reference" "#PWR07" (at 80.01 121.92 0)
-      (effects (font (size 1.27 1.27)) hide)
-    )
-    (property "Value" "GND" (at 80.137 119.9642 0)
-      (effects (font (size 1.27 1.27)))
-    )
-    (property "Footprint" "" (at 80.01 115.57 0)
-      (effects (font (size 1.27 1.27)) hide)
-    )
-    (property "Datasheet" "" (at 80.01 115.57 0)
+  (symbol (lib_id "Lily58:Jumper_NO_Small") (at 102.87 133.35 0) (unit 1)
+    (in_bom yes) (on_board yes) (dnp no)
+    (property "Reference" "JP12" (at 102.87 134.62 0)
+      (effects (font (size 1.27 1.27)))
+    )
+    (property "Value" "~" (at 102.87 130.81 0)
+      (effects (font (size 1.27 1.27)) hide)
+    )
+    (property "Footprint" "Lily58-footprint:Jumper_arrow" (at 102.87 133.35 0)
+      (effects (font (size 1.27 1.27)) hide)
+    )
+    (property "Datasheet" "~" (at 102.87 133.35 0)
+      (effects (font (size 1.27 1.27)) hide)
+    )
+    (pin "1")
+    (pin "2")
+    (instances
+      (project "Lily58_Pro"
+        (path "/f1967ba3-0d91-443c-b17c-ce0b5df5a1c7"
+          (reference "JP12") (unit 1)
+        )
+      )
+    )
+  )
+  (symbol (lib_id "Lily58:Jumper_NO_Small") (at 73.66 123.19 0) (unit 1)
+    (in_bom yes) (on_board yes) (dnp no)
+    (property "Reference" "JP1" (at 73.66 124.46 0)
+      (effects (font (size 1.27 1.27)))
+    )
+    (property "Value" "~" (at 73.66 119.38 0)
+      (effects (font (size 1.27 1.27)) hide)
+    )
+    (property "Footprint" "Lily58-footprint:Jumper_arrow" (at 73.66 123.19 0)
+      (effects (font (size 1.27 1.27)) hide)
+    )
+    (property "Datasheet" "~" (at 73.66 123.19 0)
+      (effects (font (size 1.27 1.27)) hide)
+    )
+    (pin "1")
+    (pin "2")
+    (instances
+      (project "Lily58_Pro"
+        (path "/f1967ba3-0d91-443c-b17c-ce0b5df5a1c7"
+          (reference "JP1") (unit 1)
+        )
+      )
+    )
+  )
+  (symbol (lib_id "power:GND") (at 80.01 106.68 90) (unit 1)
+    (in_bom yes) (on_board yes) (dnp no)
+    (property "Reference" "#PWR07" (at 86.36 106.68 0)
+      (effects (font (size 1.27 1.27)) hide)
+    )
+    (property "Value" "GND" (at 83.2612 106.553 90)
+      (effects (font (size 1.27 1.27)) (justify right))
+    )
+    (property "Footprint" "" (at 80.01 106.68 0)
+      (effects (font (size 1.27 1.27)) hide)
+    )
+    (property "Datasheet" "" (at 80.01 106.68 0)
       (effects (font (size 1.27 1.27)) hide)
     )
@@
         )
       )
-    )
-  )
-  (symbol (lib_id "Lily58:Jumper_NO_Small") (at 102.87 133.35 0) (unit 1)
-    (in_bom yes) (on_board yes) (dnp no)
-    (property "Reference" "JP12" (at 102.87 134.62 0)
-      (effects (font (size 1.27 1.27)))
-    )
-    (property "Value" "~" (at 102.87 130.81 0)
-      (effects (font (size 1.27 1.27)) hide)
-    )
-    (property "Footprint" "Lily58-footprint:Jumper_arrow" (at 102.87 133.35 0)
-      (effects (font (size 1.27 1.27)) hide)
-    )
-    (property "Datasheet" "~" (at 102.87 133.35 0)
-      (effects (font (size 1.27 1.27)) hide)
-    )
-    (pin "1")
-    (pin "2")
-    (instances
-      (project "Lily58_Pro"
-        (path "/f1967ba3-0d91-443c-b17c-ce0b5df5a1c7"
-          (reference "JP12") (unit 1)
-        )
-      )
-    )
-  )
-  (symbol (lib_id "Lily58:Jumper_NO_Small") (at 73.66 123.19 0) (unit 1)
-    (in_bom yes) (on_board yes) (dnp no)
-    (property "Reference" "JP1" (at 73.66 124.46 0)
-      (effects (font (size 1.27 1.27)))
-    )
-    (property "Value" "~" (at 73.66 119.38 0)
-      (effects (font (size 1.27 1.27)) hide)
-    )
-    (property "Footprint" "Lily58-footprint:Jumper_arrow" (at 73.66 123.19 0)
-      (effects (font (size 1.27 1.27)) hide)
-    )
-    (property "Datasheet" "~" (at 73.66 123.19 0)
-      (effects (font (size 1.27 1.27)) hide)
-    )
-    (pin "1")
-    (pin "2")
-    (instances
-      (project "Lily58_Pro"
-        (path "/f1967ba3-0d91-443c-b17c-ce0b5df5a1c7"
-          (reference "JP1") (unit 1)
-        )
-      )
